File: Eagle/HeaterCotrol.sch (EAGLE design)
At the start: 27 parts, among them Q1 P-FET

Commit message: Rev 1
Parts:
- removed U$9: OMROM_TH, CuriousTech:OMROM_TH
- added LEFT, RIGHT: OMROM_TH, CuriousTech:OMROM_TH
- C1: value 1uF -> 0.1uF
- R5: value 10K -> 1K
- U$8: value OMROM_TH -> SMD-PAD1; device CuriousTech:OMROM_TH -> CuriousTech:SMD-PAD1
- renumbered C3 to C1
Connections:
- net 3V3: now also U$8.P$1
- net GND: now also LEFT.P2, LEFT.P4, RIGHT.P2, RIGHT.P4; no longer U$8.P2, U$8.P4, U$9.P2, U$9.P4
- net IO13: now also RIGHT.P1; no longer U$9.P1
- net IO14: now also LEFT.P3; no longer U$8.P3
Other:
- note added: "ADC"
- note added: "DS18B20"
- note added: "Not used"
- note removed: "Temp"
- note removed: "Water Sensor"
- moved on the sheet: +, +__-, ., Q2, R2, R4, R6
