File: Eagle/HeaterCotrol.sch (EAGLE design)
At the start: 37 parts, among them J1 JUMPER_SOLDER_1X2, Q1 P-FET

Commit message: Updated for r2 board
Parts:
- removed IO12: (no value), led:LEDCHIP-LED0805
- removed J1: JUMPER_SOLDER_1X2, dp_devices:JUMPER_SOLDER_1X2
- removed R8: 10K, SparkFun-Resistors:RESISTOR0805-RES
- added C4, C5: 0.1uF, SparkFun-Capacitors:CAP
- added HEAT, IO0: (no value), led:LEDCHIP-LED0805
- added R10: 1K, SparkFun-Resistors:RESISTOR0805-RES
- added R11: 330, SparkFun-Resistors:RESISTOR0805-RES
Connections:
- removed net HEAT: Q1.B, R8.2
- removed net ICSPCLK: 10F320.GP1/AN1/ICSPCLK, R8.1, U$9.PGC
- new net N$6: Q1.B, R10.1
- new net N$7: HEAT.C, R7.2
- net 3V3: now also C4.1, C5.1, HEAT.A
- net GND: now also C4.2, C5.2, IO0.C; no longer IO12.C
- net IO0: now also R11.2
- net IO12: now also R10.2, R7.1; no longer R7.2
- net N$4: no longer J1.2
- net N$5: now also IO0.A, R11.1; no longer IO12.A, R7.1
- net REST: now also 10F320.GP1/AN1/ICSPCLK, U$9.PGC; no longer J1.1
Other:
- note added: "Optional LEDs"
- moved on the sheet: +__-, ., C1, C2, C3, FLASH, OLED, Q1, R1, R2, R3, R7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

Commit message: Extended IO0, IO2 to side
Parts:
- removed 10F320: PIC10F320T-I/OT, Microchip_By_element14_Batch_1:PIC10F220T-I/OT
- removed C3, C5: 0.1uF, SparkFun-Capacitors:CAP
- removed HEAT, IO0: (no value), led:LEDCHIP-LED0805
- removed R7: 330, SparkFun-Resistors:RESISTOR0805-RES
- added 10F: PIC10F202T-I/OT, Microchip_By_element14_Batch_1:PIC10F202T-I/OT
- added U$12, U$13, U$14: SMD-PAD1, CuriousTech:SMD-PAD1
- C4: value 0.1uF -> 1uF
- R10: value 1K -> 10K
- R11: value 330 -> 4K7
- R6: value 4K7 -> 1K
- R9: value 10K -> 4K7
- U$9: value PIC-ICSP-MINI -> SMD-PAD1; device SparkFun-Connectors:PIC-ICSP-MINI -> CuriousTech:SMD-PAD1
Connections:
- net N$3 renamed SCL
- net N$9 renamed SDA
- removed net N$5: IO0.A, R11.1
- removed net PICPWM: 10F320.GP0/AN0/ICSPDAT, R5.1, U$9.PGD
- net 3V3: now also 10F.VDD, OLED.2, R9.1, U$5.P$1, U$9.P$1; no longer 10F320.VDD, C3.1, C5.1, HEAT.A, OLED.1, R6.1, R9.2, U$4.P$1
- net ADC: now also R10.2, R11.1; no longer R4.1, U$7.P$1
- net GND: now also 10F.VSS, OLED.1, R11.2, U$13.P$1, U$4.P$1; no longer 10F320.VSS, C3.2, C5.2, IO0.C, LEFT.P2, OLED.2, U$5.P$1, U$9.GND
- net IO0: now also U$14.P$1; no longer R11.2
- net IO12: now also R5.2; no longer R10.2, R7.1
- net IO14: now also R9.2; no longer R6.2
- net IO15: now also R6.1; no longer 10F320.GP3/~MCLR/VPP, U$9.VPP
- net IO16: now also R4.1; no longer R9.1
- net IO2: now also 10F.GP0/ICSPDAT, U$12.P$1; no longer 10F320.GP2/T0CKI/FOSC4
- net N$2: now also R6.2; no longer R5.2
- net N$6: now also R5.1; no longer R10.1
- net N$7: now also R10.1, U$7.P$1; no longer HEAT.C, R7.2
- net REST: now also 10F.GP1/ICSPCLK; no longer 10F320.GP1/AN1/ICSPCLK, U$9.PGC
Other:
- note added: "Future expansion"
- note removed: "Optional LEDs"
- moved on the sheet: +, +__-, -, ., C1, C2, C4, D1, FLASH, OLED, Q1, Q2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
