File: Eagle/HeaterControlPlusPIC.brd (EAGLE design)
At the start: 25.7 x 38.1 mm, 35 parts, among them Q1 P-FET

Commit message: Update HeaterControlPlusPIC.brd
Parts:
- added R9: 10K, SparkFun-Resistors:0805
- R6: value 10K -> 4K7
- moved R4 17.8 mm to (5.59, 7.11), flipped to the bottom
- moved R6 6.86 mm to (12.2, 6.10), turned to 0 degrees
- moved U$10 4.32 mm to (10.9, 2.03)
- moved U$7 4.32 mm to (6.60, 2.03)
- moved R3 2.29 mm to (20.6, 17.0)
- moved Q1 0.51 mm to (18.5, 10.4)
- moved R2 0.25 mm to (20.6, 14.7)
Connections:
- net 3V3: now also R9.2
- net IO14: now also R6.2, U$10.>NAME; no longer LEFT.P3
- net IO16: now also LEFT.P3, R9.1; no longer R6.2, U$10.>NAME
Routing:
- net ADC: track 34.8 -> 14.0 mm
- net IO16: track 12.3 -> 6.55 mm, vias 1 -> 0
- net IO14: track 5.45 -> 11.1 mm, vias 0 -> 1
- net 3V3: track 112.4 -> 107.3 mm
- net N$22: track 22.5 -> 21.5 mm
- net HEAT: track 2.48 -> 1.98 mm
Other:
- board text added: "DS18B20 IO14"
- board text added: "IO16"
- board text removed: "DS18B20 IO16"
- board text removed: "IO14"

Commit message: Added jumper for auto-reset
Parts:
- added J1: JUMPER_SOLDER_1X2, dp_devices:JUMPER_SOLDER_1X2
Connections:
- removed net N$22: R3.1, U$1.REST
- new net REST: J1.1, R3.1, U$1.REST
- net N$4: now also J1.2
Routing:
- net REST: track 0.00 -> 24.8 mm
- net N$22: track 21.5 -> 0.00 mm
- net N$4: track 4.07 -> 14.2 mm, vias 0 -> 1
Changed lines of the file:
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@@
 <?xml version="1.0" encoding="utf-8"?>
 <!DOCTYPE eagle SYSTEM "eagle.dtd">
-<eagle version="7.4.0">
+<eagle version="7.5.0">
 <drawing>
 <settings>
@@
 <element name="C3" library="SparkFun-Capacitors" package="0805-CAP" value="0.1uF" x="12.192" y="22.86" rot="MR90"/>
 <element name="R9" library="SparkFun-Resistors" package="0805" value="10K" x="8.89" y="9.906" rot="MR90"/>
+<element name="J1" library="dp_devices" package="JUMPER_SOLDER_1X2" value="JUMPER_SOLDER_1X2" x="20.066" y="20.828" rot="R90"/>
 </elements>
 <signals>
@@
 <wire x1="14.23" y1="28.41" x2="14.23" y2="26.156" width="0.3048" layer="1"/>
 <wire x1="14.23" y1="26.156" x2="15.24" y2="25.146" width="0.3048" layer="1"/>
-<via x="15.24" y="25.146" extent="1-16" drill="0.6"/>
+<via x="15.24" y="25.146" extent="1-16" drill="0.5"/>
 <wire x1="19.674" y1="25.146" x2="15.24" y2="25.146" width="0.3048" layer="1"/>
 <contactref element="U$9" pad="1"/>
@@
 <wire x1="21.59" y1="2.032" x2="21.59" y2="8.636" width="0.6096" layer="16"/>
 <wire x1="21.59" y1="8.636" x2="19.812" y2="10.414" width="0.6096" layer="16"/>
-<via x="19.812" y="10.414" extent="1-16" drill="0.6"/>
+<via x="19.812" y="10.414" extent="1-16" drill="0.5"/>
 <wire x1="19.812" y1="10.414" x2="19.812" y2="11.568" width="0.6096" layer="1"/>
 <wire x1="19.812" y1="11.568" x2="20.182" y2="11.938" width="0.6096" layer="1"/>
@@
 <signal name="N$29">
 </signal>
-<signal name="N$22">
+<signal name="REST">
 <contactref element="R3" pad="1"/>
 <contactref element="U$1" pad="REST"/>
@@
 <wire x1="2.286" y1="14.478" x2="2.286" y2="13.1864" width="0.3048" layer="1"/>
 <wire x1="2.286" y1="13.1864" x2="2.2606" y2="13.161" width="0.3048" layer="1"/>
+<contactref element="J1" pad="1"/>
+<wire x1="19.674" y1="17.018" x2="19.674" y2="19.7756" width="0.3048" layer="1"/>
+<wire x1="19.674" y1="19.7756" x2="20.066" y2="20.1676" width="0.3048" layer="1"/>
 </signal>
 <signal name="GND">
@@
 <contactref element="U$7" pad="&gt;NAME"/>
 <wire x1="6.604" y1="2.032" x2="6.604" y2="4.572" width="0.3048" layer="16"/>
-<via x="6.604" y="4.572" extent="1-16" drill="0.6"/>
+<via x="6.604" y="4.572" extent="1-16" drill="0.5"/>
 <wire x1="6.604" y1="4.572" x2="4.23" y2="6.946" width="0.3048" layer="1"/>
 <wire x1="4.23" y1="12.51" x2="4.23" y2="6.946" width="0.3048" layer="1"/>
@@
 <wire x1="12.23" y1="28.41" x2="12.23" y2="21.298" width="0.3048" layer="1"/>
 <wire x1="12.23" y1="21.298" x2="13.208" y2="20.32" width="0.3048" layer="1"/>
-<via x="13.208" y="20.32" extent="1-16" drill="0.6"/>
+<via x="13.208" y="20.32" extent="1-16" drill="0.5"/>
 <wire x1="13.208" y1="20.32" x2="13.462" y2="20.574" width="0.3048" layer="16"/>
 <wire x1="13.462" y1="20.574" x2="14.3256" y2="20.574" width="0.3048" layer="16"/>
@@
 <wire x1="11.292" y1="6.096" x2="11.292" y2="8.266" width="0.3048" layer="16"/>
 <wire x1="11.292" y1="8.266" x2="11.176" y2="8.382" width="0.3048" layer="16"/>
-<via x="11.176" y="8.382" extent="1-16" drill="0.6"/>
+<via x="11.176" y="8.382" extent="1-16" drill="0.5"/>
 <wire x1="11.176" y1="8.382" x2="11.176" y2="9.906" width="0.3048" layer="1"/>
 <wire x1="11.176" y1="9.906" x2="10.16" y2="10.922" width="0.3048" layer="1"/>
@@
 <wire x1="19.558" y1="29.294" x2="19.558" y2="29.838" width="0.4064" layer="16"/>
 <wire x1="19.558" y1="29.838" x2="20.574" y2="30.854" width="0.4064" layer="16"/>
+<contactref element="J1" pad="2"/>
+<wire x1="20.066" y1="21.4884" x2="20.066" y2="21.844" width="0.3048" layer="1"/>
+<wire x1="20.066" y1="21.844" x2="21.59" y2="23.368" width="0.3048" layer="1"/>
+<via x="21.59" y="23.368" extent="1-16" drill="0.5"/>
+<wire x1="21.59" y1="23.368" x2="21.59" y2="28.702" width="0.3048" layer="16"/>
+<wire x1="21.59" y1="28.702" x2="21.082" y2="29.21" width="0.3048" layer="16"/>
+<wire x1="21.082" y1="29.21" x2="19.642" y2="29.21" width="0.3048" layer="16"/>
+<wire x1="19.642" y1="29.21" x2="19.558" y2="29.294" width="0.3048" layer="16"/>
 </signal>
 <signal name="N$2">
