File: Slave/WaterbedSlave.sch (EAGLE design)
At the start: 8 parts

Commit message: Update WaterbedSlave.sch
Parts:
- added LED1: (no value), led:LEDCHIPLED_0805
- added R1: 330, SparkFun-Resistors:RESISTOR0805-RES
Connections:
- new net N$10: LED1.A, R1.1
- net GND: now also LED1.C
- net N$16: now also R1.2
Other:
- moved on the sheet: JP1, U$2
Changed lines of the file:
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@@
 <part name="JP2" library="SparkFun-Connectors" deviceset="M01" device="PTH_2MM"/>
 <part name="F1" library="SparkFun-Capacitors" deviceset="CAP" device="PTH1"/>
+<part name="LED1" library="led" deviceset="LED" device="CHIPLED_0805"/>
+<part name="R1" library="SparkFun-Resistors" deviceset="RESISTOR" device="0805-RES" value="330"/>
 </parts>
 <sheets>
@@
 </plain>
 <instances>
-<instance part="U$2" gate="G$1" x="111.76" y="55.88" rot="R270"/>
-<instance part="JP1" gate="G$1" x="91.44" y="93.98" rot="R270"/>
+<instance part="U$2" gate="G$1" x="121.92" y="55.88" rot="R270"/>
+<instance part="JP1" gate="G$1" x="91.44" y="101.6" rot="R270"/>
 <instance part="C1" gate="G$1" x="83.82" y="76.2"/>
 <instance part="U$3" gate="G$1" x="17.78" y="55.88" rot="MR180"/>
@@
 <instance part="JP2" gate="G$1" x="68.58" y="33.02" rot="R90"/>
 <instance part="F1" gate="G$1" x="35.56" y="66.04" rot="R90"/>
+<instance part="LED1" gate="G$1" x="104.14" y="73.66"/>
+<instance part="R1" gate="G$1" x="104.14" y="83.82" rot="R90"/>
 </instances>
 <busses>
@@
 <pinref part="JP1" gate="G$1" pin="1"/>
 <pinref part="U$2" gate="G$1" pin="_DC-"/>
-<wire x1="88.9" y1="66.04" x2="88.9" y2="86.36" width="0.1524" layer="91"/>
-<wire x1="101.6" y1="66.04" x2="88.9" y2="66.04" width="0.1524" layer="91"/>
+<wire x1="88.9" y1="66.04" x2="88.9" y2="93.98" width="0.1524" layer="91"/>
+<wire x1="111.76" y1="66.04" x2="104.14" y2="66.04" width="0.1524" layer="91"/>
 <junction x="88.9" y="66.04"/>
 <pinref part="C1" gate="G$1" pin="-"/>
+<wire x1="104.14" y1="66.04" x2="88.9" y2="66.04" width="0.1524" layer="91"/>
 <wire x1="83.82" y1="66.04" x2="83.82" y2="71.12" width="0.1524" layer="91"/>
 <wire x1="81.28" y1="66.04" x2="83.82" y2="66.04" width="0.1524" layer="91"/>
@@
 <junction x="83.82" y="66.04"/>
 <pinref part="SUPP" gate="G$1" pin="3V3"/>
+<pinref part="LED1" gate="G$1" pin="C"/>
+<wire x1="104.14" y1="68.58" x2="104.14" y2="66.04" width="0.1524" layer="91"/>
+<junction x="104.14" y="66.04"/>
 </segment>
 </net>
@@
 <pinref part="SUPP" gate="G$1" pin="GND"/>
 <pinref part="C1" gate="G$1" pin="+"/>
-<wire x1="91.44" y1="81.28" x2="91.44" y2="86.36" width="0.1524" layer="91"/>
+<wire x1="91.44" y1="81.28" x2="91.44" y2="93.98" width="0.1524" layer="91"/>
 <wire x1="83.82" y1="78.74" x2="83.82" y2="81.28" width="0.1524" layer="91"/>
 <wire x1="83.82" y1="81.28" x2="91.44" y2="81.28" width="0.1524" layer="91"/>
@@
 <segment>
 <pinref part="JP1" gate="G$1" pin="3"/>
-<wire x1="93.98" y1="86.36" x2="93.98" y2="60.96" width="0.1524" layer="91"/>
+<wire x1="93.98" y1="93.98" x2="93.98" y2="91.44" width="0.1524" layer="91"/>
 <pinref part="U$2" gate="G$1" pin="_DC+"/>
-<wire x1="93.98" y1="60.96" x2="101.6" y2="60.96" width="0.1524" layer="91"/>
+<wire x1="93.98" y1="91.44" x2="93.98" y2="60.96" width="0.1524" layer="91"/>
+<wire x1="93.98" y1="60.96" x2="111.76" y2="60.96" width="0.1524" layer="91"/>
+<pinref part="R1" gate="G$1" pin="2"/>
+<wire x1="104.14" y1="88.9" x2="104.14" y2="91.44" width="0.1524" layer="91"/>
+<wire x1="104.14" y1="91.44" x2="93.98" y2="91.44" width="0.1524" layer="91"/>
+<junction x="93.98" y="91.44"/>
 </segment>
 </net>
@@
 <wire x1="96.52" y1="48.26" x2="96.52" y2="50.8" width="0.1524" layer="91"/>
 <pinref part="U$2" gate="G$1" pin="AC2"/>
-<wire x1="96.52" y1="50.8" x2="101.6" y2="50.8" width="0.1524" layer="91"/>
+<wire x1="96.52" y1="50.8" x2="111.76" y2="50.8" width="0.1524" layer="91"/>
 <pinref part="U$3" gate="G$1" pin="H"/>
 <wire x1="22.86" y1="55.88" x2="25.4" y2="55.88" width="0.1524" layer="91"/>
@@
 <segment>
 <pinref part="U$2" gate="G$1" pin="AC1"/>
-<wire x1="101.6" y1="43.18" x2="68.58" y2="43.18" width="0.1524" layer="91"/>
+<wire x1="111.76" y1="43.18" x2="68.58" y2="43.18" width="0.1524" layer="91"/>
 <wire x1="68.58" y1="43.18" x2="68.58" y2="40.64" width="0.1524" layer="91"/>
 <pinref part="JP2" gate="G$1" pin="1"/>
@@
 </segment>
 </net>
+<net name="N$10" class="0">
+<segment>
+<pinref part="R1" gate="G$1" pin="1"/>
+<pinref part="LED1" gate="G$1" pin="A"/>
+<wire x1="104.14" y1="78.74" x2="104.14" y2="76.2" width="0.1524" layer="91"/>
+</segment>
+</net>

Commit message: New cheap model
Parts:
- removed C1: 330uF, resistor:CPOL-USTT5D9
- removed SUPP: RAC02-3.3SC, CuriousTech:RAC02-3.3SC
- added R2: 330, SparkFun-Resistors:RESISTOR0805-RES
- added SSR: IXYS CPC1998J, CuriousTech:SSR-5A-240VACI4-PAC
- U$2: value SSR-5A-240VAC -> 3V3AC-DC; device CuriousTech:SSR-5A-240VAC -> CuriousTech:RAC02-3.3SCCHEAP
- renumbered JP2 to O2, JP3 to O1, LED1 to LED
Connections:
- removed net N$14: SUPP.AC2, U$2.AC2, U$3.H
- new net N$2: F1.2, U$2.AC2
- new net N$3: O2.1, SSR.AC2
- net GND: now also SSR._DC-, U$2.3V3; no longer C1.-, SUPP.3V3, U$2._DC-
- net N$1: now also U$2.AC1; no longer F1.1
- net N$15: now also U$2.GND; no longer C1.+, SUPP.GND
- net N$16: now also R2.1; no longer U$2._DC+
- net N$5: now also R2.2, SSR._DC+; no longer F1.2, SUPP.AC1
- net N$6: now also F1.1, SSR.AC1, U$3.H; no longer O2.1, U$2.AC1
Other:
- moved on the sheet: F1, U$2
Changed lines of the file:
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@@
 <?xml version="1.0" encoding="utf-8"?>
 <!DOCTYPE eagle SYSTEM "eagle.dtd">
-<eagle version="7.5.0">
+<eagle version="9.1.1">
 <drawing>
 <settings>
 <setting alwaysvectorfont="no"/>
+<setting keepoldvectorfont="yes"/>
 <setting verticaltext="up"/>
 </settings>
@@
 <layer number="112" name="tSilk" color="7" fill="1" visible="yes" active="yes"/>
 <layer number="113" name="IDFDebug" color="7" fill="1" visible="yes" active="yes"/>
+<layer number="114" name="Badge_Outline" color="7" fill="1" visible="yes" active="yes"/>
+<layer number="115" name="ReferenceISLANDS" color="7" fill="1" visible="yes" active="yes"/>
 <layer number="116" name="Patch_BOT" color="9" fill="4" visible="yes" active="yes"/>
 <layer number="118" name="Rect_Pads" color="7" fill="1" visible="yes" active="yes"/>
@@
 </classes>
 <parts>
-<part name="U$2" library="CuriousTech" deviceset="SSR-5A-240VAC" device=""/>
 <part name="JP1" library="SparkFun-Connectors" deviceset="M03" device="POLAR_LOCK"/>
-<part name="C1" library="resistor" deviceset="CPOL-US" device="TT5D9" value="330uF"/>
 <part name="U$3" library="CuriousTech" deviceset="IEC" device="" value="IEC 0714-7-E"/>
-<part name="SUPP" library="CuriousTech" deviceset="RAC02-3.3SC" device=""/>
-<part name="JP3" library="SparkFun-Connectors" deviceset="M01" device="PTH_2MM"/>
-<part name="JP2" library="SparkFun-Connectors" deviceset="M01" device="PTH_2MM"/>
+<part name="O1" library="SparkFun-Connectors" deviceset="M01" device="PTH_2MM"/>
+<part name="O2" library="SparkFun-Connectors" deviceset="M01" device="PTH_2MM"/>
 <part name="F1" library="SparkFun-Capacitors" deviceset="CAP" device="PTH1"/>
-<part name="LED1" library="led" deviceset="LED" device="CHIPLED_0805"/>
+<part name="LED" library="led" deviceset="LED" device="CHIPLED_0805"/>
 <part name="R1" library="SparkFun-Resistors" deviceset="RESISTOR" device="0805-RES" value="330"/>
+<part name="SSR" library="CuriousTech" deviceset="SSR-5A-240VAC" device="I4-PAC" value="IXYS CPC1998J"/>
+<part name="U$2" library="CuriousTech" deviceset="RAC02-3.3SC" device="CHEAP" value="3V3AC-DC"/>
+<part name="R2" library="SparkFun-Resistors" deviceset="RESISTOR" device="0805-RES" value="330"/>
 </parts>
 <sheets>
@@
 </plain>
 <instances>
-<instance part="U$2" gate="G$1" x="121.92" y="55.88" rot="R270"/>
 <instance part="JP1" gate="G$1" x="91.44" y="101.6" rot="R270"/>
-<instance part="C1" gate="G$1" x="83.82" y="76.2"/>
 <instance part="U$3" gate="G$1" x="17.78" y="55.88" rot="MR180"/>
-<instance part="SUPP" gate="G$1" x="60.96" y="60.96"/>
-<instance part="JP3" gate="G$1" x="60.96" y="33.02" rot="R90"/>
-<instance part="JP2" gate="G$1" x="68.58" y="33.02" rot="R90"/>
-<instance part="F1" gate="G$1" x="35.56" y="66.04" rot="R90"/>
-<instance part="LED1" gate="G$1" x="104.14" y="73.66"/>
+<instance part="O1" gate="G$1" x="60.96" y="33.02" rot="R90"/>
+<instance part="O2" gate="G$1" x="68.58" y="33.02" rot="R90"/>
+<instance part="F1" gate="G$1" x="35.56" y="55.88" rot="R90"/>
+<instance part="LED" gate="G$1" x="104.14" y="73.66"/>
 <instance part="R1" gate="G$1" x="104.14" y="83.82" rot="R90"/>
+<instance part="SSR" gate="G$1" x="124.46" y="55.88" rot="R270"/>
+<instance part="U$2" gate="G$1" x="60.96" y="60.96"/>
+<instance part="R2" gate="G$1" x="106.68" y="60.96"/>
 </instances>
 <busses>
@@
 <segment>
 <pinref part="JP1" gate="G$1" pin="1"/>
-<pinref part="U$2" gate="G$1" pin="_DC-"/>
 <wire x1="88.9" y1="66.04" x2="88.9" y2="93.98" width="0.1524" layer="91"/>
-<wire x1="111.76" y1="66.04" x2="104.14" y2="66.04" width="0.1524" layer="91"/>
 <junction x="88.9" y="66.04"/>
-<pinref part="C1" gate="G$1" pin="-"/>
 <wire x1="104.14" y1="66.04" x2="88.9" y2="66.04" width="0.1524" layer="91"/>
-<wire x1="83.82" y1="66.04" x2="83.82" y2="71.12" width="0.1524" layer="91"/>
 <wire x1="81.28" y1="66.04" x2="83.82" y2="66.04" width="0.1524" layer="91"/>
 <wire x1="83.82" y1="66.04" x2="88.9" y2="66.04" width="0.1524" layer="91"/>
-<junction x="83.82" y="66.04"/>
-<pinref part="SUPP" gate="G$1" pin="3V3"/>
-<pinref part="LED1" gate="G$1" pin="C"/>
+<pinref part="LED" gate="G$1" pin="C"/>
 <wire x1="104.14" y1="68.58" x2="104.14" y2="66.04" width="0.1524" layer="91"/>
+<wire x1="104.14" y1="66.04" x2="111.76" y2="66.04" width="0.1524" layer="91"/>
 <junction x="104.14" y="66.04"/>
+<wire x1="111.76" y1="66.04" x2="114.3" y2="66.04" width="0.1524" layer="91"/>
+<pinref part="SSR" gate="G$1" pin="_DC-"/>
+<pinref part="U$2" gate="G$1" pin="3V3"/>
 </segment>
 </net>
@@
 <pinref part="JP1" gate="G$1" pin="2"/>
 <wire x1="91.44" y1="60.96" x2="91.44" y2="81.28" width="0.1524" layer="91"/>
-<pinref part="SUPP" gate="G$1" pin="GND"/>
-<pinref part="C1" gate="G$1" pin="+"/>
 <wire x1="91.44" y1="81.28" x2="91.44" y2="93.98" width="0.1524" layer="91"/>
-<wire x1="83.82" y1="78.74" x2="83.82" y2="81.28" width="0.1524" layer="91"/>
-<wire x1="83.82" y1="81.28" x2="91.44" y2="81.28" width="0.1524" layer="91"/>
-<junction x="91.44" y="81.28"/>
+<pinref part="U$2" gate="G$1" pin="GND"/>
 </segment>
 </net>
@@
 <pinref part="JP1" gate="G$1" pin="3"/>
 <wire x1="93.98" y1="93.98" x2="93.98" y2="91.44" width="0.1524" layer="91"/>
-<pinref part="U$2" gate="G$1" pin="_DC+"/>
 <wire x1="93.98" y1="91.44" x2="93.98" y2="60.96" width="0.1524" layer="91"/>
-<wire x1="93.98" y1="60.96" x2="111.76" y2="60.96" width="0.1524" layer="91"/>
 <pinref part="R1" gate="G$1" pin="2"/>
 <wire x1="104.14" y1="88.9" x2="104.14" y2="91.44" width="0.1524" layer="91"/>
 <wire x1="104.14" y1="91.44" x2="93.98" y2="91.44" width="0.1524" layer="91"/>
 <junction x="93.98" y="91.44"/>
-</segment>
-</net>
-<net name="N$14" class="0">
-<segment>
-<wire x1="25.4" y1="55.88" x2="25.4" y2="48.26" width="0.1524" layer="91"/>
-<wire x1="25.4" y1="48.26" x2="96.52" y2="48.26" width="0.1524" layer="91"/>
-<wire x1="96.52" y1="48.26" x2="96.52" y2="50.8" width="0.1524" layer="91"/>
-<pinref part="U$2" gate="G$1" pin="AC2"/>
-<wire x1="96.52" y1="50.8" x2="111.76" y2="50.8" width="0.1524" layer="91"/>
-<pinref part="U$3" gate="G$1" pin="H"/>
-<wire x1="22.86" y1="55.88" x2="25.4" y2="55.88" width="0.1524" layer="91"/>
-<pinref part="SUPP" gate="G$1" pin="AC2"/>
-<wire x1="25.4" y1="55.88" x2="40.64" y2="55.88" width="0.1524" layer="91"/>
-<junction x="25.4" y="55.88"/>
+<pinref part="R2" gate="G$1" pin="1"/>
+<wire x1="93.98" y1="60.96" x2="101.6" y2="60.96" width="0.1524" layer="91"/>
 </segment>
 </net>
@@
 <wire x1="0" y1="81.28" x2="27.94" y2="81.28" width="0.1524" layer="91"/>
 <wire x1="27.94" y1="81.28" x2="27.94" y2="66.04" width="0.1524" layer="91"/>
-<pinref part="JP3" gate="G$1" pin="1"/>
+<pinref part="O1" gate="G$1" pin="1"/>
+<pinref part="U$2" gate="G$1" pin="AC1"/>
+<wire x1="27.94" y1="66.04" x2="40.64" y2="66.04" width="0.1524" layer="91"/>
+<junction x="27.94" y="66.04"/>
+</segment>
+</net>
+<net name="N$10" class="0">
+<segment>
+<pinref part="R1" gate="G$1" pin="1"/>
+<pinref part="LED" gate="G$1" pin="A"/>
+<wire x1="104.14" y1="78.74" x2="104.14" y2="76.2" width="0.1524" layer="91"/>
+</segment>
+</net>
+<net name="N$2" class="0">
+<segment>
+<pinref part="F1" gate="G$1" pin="2"/>
+<pinref part="U$2" gate="G$1" pin="AC2"/>
+<wire x1="38.1" y1="55.88" x2="40.64" y2="55.88" width="0.1524" layer="91"/>
+</segment>
+</net>
+<net name="N$3" class="0">
+<segment>
+<wire x1="68.58" y1="43.18" x2="68.58" y2="40.64" width="0.1524" layer="91"/>
+<pinref part="O2" gate="G$1" pin="1"/>
+<wire x1="68.58" y1="43.18" x2="93.98" y2="43.18" width="0.1524" layer="91"/>
+<wire x1="93.98" y1="43.18" x2="93.98" y2="50.8" width="0.1524" layer="91"/>
+<pinref part="SSR" gate="G$1" pin="AC2"/>
+<wire x1="93.98" y1="50.8" x2="114.3" y2="50.8" width="0.1524" layer="91"/>
+</segment>
+</net>
+<net name="N$6" class="0">
+<segment>
+<wire x1="25.4" y1="55.88" x2="25.4" y2="48.26" width="0.1524" layer="91"/>
+<wire x1="25.4" y1="48.26" x2="96.52" y2="48.26" width="0.1524" layer="91"/>
+<pinref part="U$3" gate="G$1" pin="H"/>
+<wire x1="22.86" y1="55.88" x2="25.4" y2="55.88" width="0.1524" layer="91"/>
 <pinref part="F1" gate="G$1" pin="1"/>
-<wire x1="30.48" y1="66.04" x2="27.94" y2="66.04" width="0.1524" layer="91"/>
-<junction x="27.94" y="66.04"/>
-</segment>
-</net>
-<net name="N$6" class="0">
-<segment>
-<pinref part="U$2" gate="G$1" pin="AC1"/>
-<wire x1="111.76" y1="43.18" x2="68.58" y2="43.18" width="0.1524" layer="91"/>
-<wire x1="68.58" y1="43.18" x2="68.58" y2="40.64" width="0.1524" layer="91"/>
-<pinref part="JP2" gate="G$1" pin="1"/>
+<wire x1="25.4" y1="55.88" x2="30.48" y2="55.88" width="0.1524" layer="91"/>
+<junction x="25.4" y="55.88"/>
+<wire x1="96.52" y1="48.26" x2="106.68" y2="48.26" width="0.1524" layer="91"/>
+<wire x1="106.68" y1="48.26" x2="106.68" y2="43.18" width="0.1524" layer="91"/>
+<wire x1="111.76" y1="43.18" x2="114.3" y2="43.18" width="0.1524" layer="91"/>
+<pinref part="SSR" gate="G$1" pin="AC1"/>
+<wire x1="106.68" y1="43.18" x2="111.76" y2="43.18" width="0.1524" layer="91"/>
 </segment>
 </net>
 <net name="N$5" class="0">
 <segment>
-<pinref part="F1" gate="G$1" pin="2"/>
-<pinref part="SUPP" gate="G$1" pin="AC1"/>
-<wire x1="38.1" y1="66.04" x2="40.64" y2="66.04" width="0.1524" layer="91"/>
-</segment>
-</net>
-<net name="N$10" class="0">
-<segment>
-<pinref part="R1" gate="G$1" pin="1"/>
-<pinref part="LED1" gate="G$1" pin="A"/>
-<wire x1="104.14" y1="78.74" x2="104.14" y2="76.2" width="0.1524" layer="91"/>
-</segment>
-</net>
+<pinref part="SSR" gate="G$1" pin="_DC+"/>
+<wire x1="111.76" y1="60.96" x2="114.3" y2="60.96" width="0.1524" layer="91"/>
+<pinref part="R2" gate="G$1" pin="2"/>
+</segment>
+</net>
